Commit message: Working state

File: ses_ws/src/rotors_simulator/rotors_description/urdf/firefly_base.xacro (robot description, xacro)
@@ -41,3 +41,9 @@
       wait_to_record_bag="$(arg wait_to_record_bag)" />
   </xacro:if>
+  <xacro:arg name="gpu" default="true"/>
+  <xacro:property name="gpu" value="$(arg gpu)" />
+  <xacro:include filename="$(find velodyne_description)/urdf/VLP-16.urdf.xacro"/>
+  <VLP-16 parent="${namespace}/base_link" name="${namespace}/velodyne" topic="/velodyne_points" hz="60" samples="440" gpu="${gpu}">
+    <origin xyz="0 0 0.1" rpy="0 0 0" />
+  </VLP-16>
 </robot>

File: ses_ws/src/velodyne_simulator/velodyne_description/urdf/VLP-16.urdf.xacro (robot description, xacro)
@@ -10,9 +10,9 @@
     <link name="${name}_base_link">
       <inertial>
-        <mass value="0.83"/>
+        <mass value="0.01"/>
         <origin xyz="0 0 0.03585"/>
-        <inertia ixx="${(0.83 * (3.0*0.0516*0.0516 + 0.0717*0.0717)) / 12.0}" ixy="0" ixz="0"
-          iyy="${(0.83 * (3.0*0.0516*0.0516 + 0.0717*0.0717)) / 12.0}" iyz="0"
-          izz="${0.5 * 0.83 * (0.0516*0.0516)}"/>
+        <inertia ixx="0.01" ixy="0" ixz="0"
+          iyy="0.01" iyz="0"
+          izz="0.01"/>
       </inertial>
       <visual>

Commit message: added camera pluguin

File: ses_ws/src/rotors_simulator/rotors_description/urdf/firefly_base.xacro (robot description, xacro)
@@ -47,3 +47,21 @@
     <origin xyz="0 0 0.1" rpy="0 0 0" />
   </VLP-16>
+    <xacro:camera_macro
+    namespace="${namespace}"
+    parent_link="${namespace}/base_link"
+    camera_suffix="red_iris"
+    frame_rate="30.0"
+    horizontal_fov="1.3962634"
+    image_width="800"
+    image_height="800"
+    image_format="R8G8B8"
+    min_distance="0.02"
+    max_distance="300"
+    noise_mean="0.0"
+    noise_stddev="0.007"
+    enable_visual="1"
+    >
+    <box size="0.05 0.05 0.05" />
+    <origin xyz="0 0 0.2" rpy="0 0 0"/>
+    </xacro:camera_macro>
 </robot>
